File: PCB/motherboard/connectors.kicad_sch (KiCad schematic)
At the start: 0 parts

Commit message: test kicad collab
Parts:
- added J1: Conn_01x07_Socket, symbol Connector:Conn_01x07_Socket
Changed lines of the file:
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@@
 		(rev "0")
 	)
+	(symbol
+		(lib_id "Connector:Conn_01x07_Socket")
+		(at 107.95 52.07 0)
+		(unit 1)
+		(exclude_from_sim no)
+		(in_bom yes)
+		(on_board yes)
+		(dnp no)
+		(fields_autoplaced yes)
+		(property "Reference" "J1"
+			(at 109.22 50.7999 0)
+			(effects
+				(font
+					(size 1.27 1.27)
+				)
+				(justify left)
+			)
+		)
+		(property "Value" "Conn_01x07_Socket"
+			(at 109.22 53.3399 0)
+			(effects
+				(font
+					(size 1.27 1.27)
+				)
+				(justify left)
+			)
+		)
+		(property "Footprint" ""
+			(at 107.95 52.07 0)
+			(effects
+				(font
+					(size 1.27 1.27)
+				)
+				(hide yes)
+			)
+		)
+		(property "Datasheet" "~"
+			(at 107.95 52.07 0)
+			(effects
+				(font
+					(size 1.27 1.27)
+				)
+				(hide yes)
+			)
+		)
+		(property "Description" "Generic connector, single row, 01x07, script generated"
+			(at 107.95 52.07 0)
+			(effects
+				(font
+					(size 1.27 1.27)
+				)
+				(hide yes)
+			)
+		)
+		(pin "3"
+		)
+		(pin "6"
+		)
+		(pin "1"
+		)
+		(pin "2"
+		)
+		(pin "4"
+		)
+		(pin "5"
+		)
+		(pin "7"
+		)
+		(instances
+			(project ""
+				(path "/932efb2d-d041-4add-96d0-4fa635c69d39/85256a3a-9f5b-49e7-815e-3032a2c93bab"
+					(reference "J1")
+					(unit 1)
+				)
+			)
+		)
+	)
 )

Commit message: layout connettori + note
Parts:
- removed J1: Conn_01x07_Socket, symbol Connector:Conn_01x07_Socket
- added J1: Conn_01x04, symbol Connector_Generic:Conn_01x04
- added J2: Conn_01x08, symbol Connector_Generic:Conn_01x08
- added J3: Conn_01x06, symbol Connector_Generic:Conn_01x06
- added J4, J5: Conn_01x03, symbol Connector_Generic:Conn_01x03
- added J6: Conn_01x02, symbol Connector_Generic:Conn_01x02
- added J7: Screw_Terminal_01x03, symbol Connector:Screw_Terminal_01x03
- added J8: Screw_Terminal_01x09, symbol Connector:Screw_Terminal_01x09
- added J9: Conn_01x11, symbol Connector_Generic:Conn_01x11
Connections:
- new net +24V: J6.1 (Pin_1)
- new net +3.3V: J1.2 (Pin_2), J3.5 (Pin_5), J4.1 (Pin_1), J5.1 (Pin_1)
- new net +5V: J2.8 (Pin_8), J8.6 (Pin_6)
- new net A_IN_2_+: J9.3 (Pin_3)
- new net A_IN_2_-: J9.4 (Pin_4)
- new net A_OUT_1: J9.5 (Pin_5)
- new net A_OUT_2: J9.6 (Pin_6)
- new net D-IN_2: J9.9 (Pin_9)
- new net D_IN_1: J9.8 (Pin_8)
- new net D_IN_3: J9.10 (Pin_10)
- new net D_IN_4: J9.11 (Pin_11)
- new net ENCH_CH_A\: J8.2 (Pin_2)
- new net ENC_A: J2.2 (Pin_2)
- new net ENC_A\: J2.1 (Pin_1)
- new net ENC_B: J2.4 (Pin_4)
- new net ENC_B\: J2.3 (Pin_3)
- new net ENC_CH_A: J8.1 (Pin_1)
- new net ENC_CH_B: J8.3 (Pin_3)
- new net ENC_CH_B\: J8.4 (Pin_4)
- new net ENC_Z: J2.6 (Pin_6)
- new net ENC_Z\: J2.5 (Pin_5)
- new net GND: J1.3 (Pin_3), J2.7 (Pin_7), J3.3 (Pin_3), J3.6 (Pin_6), J4.3 (Pin_3), J5.3 (Pin_3), J6.2 (Pin_2), J8.5 (Pin_5), J9.2 (Pin_2), J9.7 (Pin_7)
- new net H1: J8.7 (Pin_7)
- new net H2: J8.8 (Pin_8)
- new net H3: J8.9 (Pin_9)
- new net MW1_motor: J7.1 (Pin_1)
- new net MW2_motor: J7.2 (Pin_2)
- new net MW3_motor: J7.3 (Pin_3)
- new net PWM: J9.1 (Pin_1)
- new net SCL: J1.1 (Pin_1), J3.4 (Pin_4)
- new net SDA: J1.4 (Pin_4), J3.2 (Pin_2)
- new net SW_1: J4.2 (Pin_2)
- new net SW_2: J5.2 (Pin_2)
Other:
- note added: "DBS36/50"
- note added: "ESCON"
- note added: "POWER CONN"
- note added: "SDP8xx-Digital"
- note added: "SFM3304-xxx-D"
- note added: "SWITCH 1"
- note added: "SWITCH 2"
