File: PCB/motherboard/ESCON50_5_sch.kicad_sch (KiCad schematic)
At the start: 27 parts, among them Q1 NMOS, Q2 PMOS, U6 LM74700QDBVTQ1, U9 TL431D

Commit message: added last footprint on sch
Parts:
- L2, L3, L4: footprint induttorejlpcb_escon:Senza-titolo -> inductors:IND-SMD_L17.0-W17.0_YSPIA1770-100M
- Q1: footprint (none) -> transistors:PG-TDSON-8_L5.0-W6.0-P1.27-BL-EP
- Q2: footprint (none) -> transistors:DFN-8_L5.7-W4.9-P1.27-LS6.1-BL
- R28: footprint (none) -> resistors:TO-220-2_L10.1-W4.5-P5.08-L
- U9: footprint Package_SO:SOIC-8_3.9x4.9mm_P1.27mm -> diodes:SOT-23-3_L2.9-W1.5-P1.90-LS2.6-BR
Changed lines of the file:
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@@
 			)
 		)
-		(property "Footprint" "induttorejlpcb_escon:Senza-titolo"
+		(property "Footprint" "inductors:IND-SMD_L17.0-W17.0_YSPIA1770-100M"
 			(at 59.69 206.68 0)
 			(hide yes)
@@
 			)
 		)
-		(property "Footprint" ""
+		(property "Footprint" "transistors:PG-TDSON-8_L5.0-W6.0-P1.27-BL-EP"
 			(at 172.72 54.61 0)
 			(hide yes)
@@
 			)
 		)
-		(property "Footprint" ""
+		(property "Footprint" "resistors:TO-220-2_L10.1-W4.5-P5.08-L"
 			(at 266.192 101.6 90)
 			(hide yes)
@@
 			)
 		)
-		(property "Footprint" "Package_SO:SOIC-8_3.9x4.9mm_P1.27mm"
+		(property "Footprint" "diodes:SOT-23-3_L2.9-W1.5-P1.90-LS2.6-BR"
 			(at 257.81 104.14 0)
 			(hide yes)
@@
 			)
 		)
-		(property "Footprint" "induttorejlpcb_escon:Senza-titolo"
+		(property "Footprint" "inductors:IND-SMD_L17.0-W17.0_YSPIA1770-100M"
 			(at 57.15 234.62 0)
 			(hide yes)
@@
 			)
 		)
-		(property "Footprint" "induttorejlpcb_escon:Senza-titolo"
+		(property "Footprint" "inductors:IND-SMD_L17.0-W17.0_YSPIA1770-100M"
 			(at 57.15 263.83 0)
 			(hide yes)
@@
 			)
 		)
-		(property "Footprint" ""
+		(property "Footprint" "transistors:DFN-8_L5.7-W4.9-P1.27-LS6.1-BL"
 			(at 270.51 92.71 0)
 			(hide yes)

Commit message: pcb layout
Parts:
- removed U9: TL431D, diodes:SOT-23-3_L2.9-W1.5-P1.90-LS2.6-BR, symbol Reference_Voltage:TL431D
- added U9: TL431AIDR, TL431AIDR:D8, symbol TL431AIDR:TL431AIDR
- C15, C16, C17, C18, C19, C20, C21, C22, C23, C24: VRATE (none) -> 50
Connections:
- net GND: now also U9.2 (ANODE), U9.3 (ANODE), U9.6 (ANODE), U9.7 (ANODE)
- net at R27.2: now also U9.1 (CATHODE)
- net at R23.2, R24.1: now also U9.8 (REF)
Other:
- moved on the sheet: C15, C16, C17, C18, C19, C20, C21, C22, C23, C24, E1, L2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
