File: PCB/motherboard/motherboard.kicad_sch (KiCad schematic)
At the start: 0 parts

Commit message: pcb layout
Parts:
- added H1, H2, H3, H4: MountingHole, MountingHole:MountingHole_3.2mm_M3, symbol Mechanical:MountingHole
