File: PCB/motherboard/motherboard.kicad_pcb (KiCad board)
At the start: 4 copper layers, 148.8 x 100 mm, 111 parts, among them J1 Conn_01x04, J10 Screw_Terminal_01x03, J11 Conn_01x05, J12 Conn_01x11, J13 Conn_01x03, J2 Conn_01x06, J3 Conn_01x08, J4 Conn_01x04, J5 Conn_01x03, J6 Conn_01x03, J8 Conn_01x06, J9 Conn_01x02, Q1 NMOS, Q2 PMOS, Q3 NMOS, U1 TPS54140ADGQR, U2 PTPS259830LNRGER, U3 AP2112K-3.3TRG1, U4 NUCLEO-L432KC, U5 TXS0104EPWR, U6 LM74700QDBVTQ1, U7 25LC256-I/SN, U8 AM26LS32ACDR, U9 TL431AIDR

Commit message: motherboard PCB rev2
Routing:
- net GND: track 27.6 -> 22.7 mm, vias 26 -> 366
- net +5V: track 20.4 -> 18.6 mm, vias 43 -> 42
- net (no net): vias 0 -> 1
Other:
- board text added: "MADE IN POLIMI BY GRUPPO VIOLA"
- board text removed: "MADE IN POLIMI BY GRUPPO VIOLA (VETERANI DEL SALTO)"
