File: PCB/motherboard/bckup/bckup.kicad_sch (KiCad schematic)
At the start: 9 parts, among them J1 Conn_01x04, J2 Conn_01x08, J3 Conn_01x06, J4 Conn_01x03, J5 Conn_01x03, J6 Conn_01x02, J7 Screw_Terminal_01x03, J8 Screw_Terminal_01x09, J9 Conn_01x11

Commit message: match label
Connections:
- net ENC_A: no longer J8.1 (Pin_1)
- net ENC_B: no longer J8.3 (Pin_3)
- net ENC_B\: no longer J8.4 (Pin_4)
- net A_IN_2+ renamed A_IN_2_+
- net A_IN_2- renamed A_IN_2_-
- net D_IN_2 renamed D-IN_2
- net D_IN_OUT_3 renamed D_IN_3
- net D_IN_OUT_4 renamed D_IN_4
- net ENCH_A\ renamed ENCH_CH_A\
- net PWM_ESCON renamed PWM
- new net ENC_CH_A: J8.1 (Pin_1)
- new net ENC_CH_B: J8.3 (Pin_3)
- new net ENC_CH_B\: J8.4 (Pin_4)
Other:
- title: CONNECTORS -> (none)
- moved on the sheet: J1, J2, J3, J4, J5, J6, J7, J8, J9
